Commit message: Bind HOIDiNi stage 2 to shared scene

File: tests/fixtures/hoidini_intermimic/asset3d/red_mug/result/red_mug.urdf (robot description, URDF)
Before this commit: robot mug, 1 links, 0 joints
Links:
- removed link mug
- added link red_mug, mass 0.35; collision mesh filename=mesh/red_mug_collision.obj scale=1 1 1; visual mesh filename=mesh/red_mug.obj scale=1 1 1
